Commit message: Next up: Setting up Odometry

File: ackermann_v2/src/description/ackermann_robot_description.urdf (robot description, URDF)
Before this commit: robot ackermann_v2, 4 links, 3 joints
Links:
- removed link imu_link
- link base_link: geometry collision box size=${base_length} ${base_width} ${base_height}; visual box size=${base_length} ${base_width} ${base_height}
- link front_caster: geometry collision sphere radius=${(wheel_radius+wheel_zoff-(base_height/2))}; visual sphere radius=${(wheel_radius+wheel_zoff-(base_height/2))}
Joints:
- removed joint imu_joint
