Commit message: The same as below

File: ackermann_v2/src/description/ackermann_vehicle.urdf (robot description, URDF)
Before this commit: robot ackermann_vehicle, 9 links, 8 joints
Links:
- removed link lidar_base
- removed link odom
- added link base_footprint
- added link lidar_link, mass 1.0; collision cylinder length=0.05 radius=0.05; visual cylinder length=0.05 radius=0.05
- link base_link: geometry collision box size=0.5 0.3 0.15; visual box size=0.5 0.3 0.15
- link wheel_back_left: geometry collision sphere radius=0.10; visual cylinder length=0.05 radius=0.10
- link wheel_back_right: geometry collision sphere radius=0.10; visual cylinder length=0.05 radius=0.10
- link wheel_front_left: geometry collision sphere radius=0.10; visual cylinder length=0.05 radius=0.10
- link wheel_front_right: geometry collision sphere radius=0.10; visual cylinder length=0.05 radius=0.10
Joints:
- removed joint odom_joint
- added joint base_joint: type fixed, parent base_link, child base_footprint, origin xyz=0.0 0.0 -0.2 rpy=0 0 0
- joint left_steering_joint: origin xyz=0.5 0.4 0.0 rpy=0 0 0 -> xyz=0.25 0.2 -0.1 rpy=0 0 0
- joint lidar_joint: child lidar_base -> lidar_link; origin xyz=0.0 0.0 0.2 rpy=0 0 0 -> xyz=0.0 0.0 0.1 rpy=0 0 0
- joint rear_left_joint: origin xyz=-0.5 0.4 0.0 rpy=1.57 0 0 -> xyz=-0.25 0.2 -0.1 rpy=1.57 0 0
- joint rear_right_joint: origin xyz=-0.5 -0.4 0.0 rpy=1.57 0 0 -> xyz=-0.25 -0.2 -0.1 rpy=1.57 0 0
- joint right_steering_joint: origin xyz=0.5 -0.4 0.0 rpy=0 0 0 -> xyz=0.25 -0.2 -0.1 rpy=0 0 0

Commit message: Car scaled, model working with nav2 example, humor gitówa

File: ackermann_v2/src/description/ackermann_vehicle.urdf (robot description, URDF)
Before this commit: robot ackermann_vehicle, 9 links, 8 joints
Links:
- link base_link: geometry collision box size=0.2 0.1 0.15; visual box size=0.2 0.1 0.06
- link lidar_link: geometry collision cylinder length=0.01 radius=0.02; visual cylinder length=0.01 radius=0.02
- link wheel_back_left: geometry collision sphere radius=0.08; visual cylinder length=0.02 radius=0.08
- link wheel_back_right: geometry collision sphere radius=0.08; visual cylinder length=0.02 radius=0.08
- link wheel_front_left: geometry collision sphere radius=0.08; visual cylinder length=0.02 radius=0.08
- link wheel_front_right: geometry collision sphere radius=0.08; visual cylinder length=0.02 radius=0.08
Joints:
- joint base_joint: origin xyz=0.0 0.0 -0.2 rpy=0 0 0 -> xyz=0.0 0.0 -0.05 rpy=0 0 0
- joint left_steering_joint: origin xyz=0.25 0.2 -0.1 rpy=0 0 0 -> xyz=0.1 0.06 -0.03 rpy=0 0 0
- joint lidar_joint: origin xyz=0.0 0.0 0.1 rpy=0 0 0 -> xyz=0.0 0.0 0.05 rpy=0 0 0
- joint rear_left_joint: origin xyz=-0.25 0.2 -0.1 rpy=1.57 0 0 -> xyz=-0.1 0.06 -0.03 rpy=1.57 0 0
- joint rear_right_joint: origin xyz=-0.25 -0.2 -0.1 rpy=1.57 0 0 -> xyz=-0.1 -0.06 -0.03 rpy=1.57 0 0
- joint right_steering_joint: origin xyz=0.25 -0.2 -0.1 rpy=0 0 0 -> xyz=0.1 -0.06 -0.03 rpy=0 0 0

Commit message: Fix vehicle footprint, add MPPI and HybridPlanner

File: ackermann_v2/src/description/ackermann_vehicle.urdf (robot description, URDF)
Before this commit: robot ackermann_vehicle, 9 links, 8 joints
Joints:
- joint base_joint: origin xyz=0.0 0.0 -0.05 rpy=0 0 0 -> xyz=-0.1 0.0 -0.05 rpy=0 0 0
